Commit message: update chassi

File: description/robot_core.xacro (robot description, xacro)
@@ -24,9 +24,9 @@
         <parent link="base_link"/>
         <child link="chassis"/>
-        <origin xyz="-0.07 0 0" />
+        <origin xyz="-0.05 0 0" />
     </joint>
     <link name="chassis">
         <visual>
-            <origin xyz="0.15 0 0.075" />
+            <origin xyz="0.10 0 0.075" />
             <geometry>
                 <box size="0.27 0.2 0.17"/>
@@ -41,5 +41,5 @@
         </collision>
         <xacro:inertial_box mass="0.5" x="0.27" y="0.2" z="0.17" >
-            <origin xyz="0.15 0 0.075" rpy="0 0 0"/>
+            <origin xyz="0.10 0 0.075" rpy="0 0 0"/>
         </xacro:inertial_box>
     </link>

Commit message: update slam

File: description/robot_core.xacro (robot description, xacro)
@@ -19,4 +19,12 @@
     <!-- Base Link -->
     <link name="base_link" >
+    </link>
+      <!-- BASE_FOOTPRINT LINK -->
+    <joint name="base_footprint_joint" type="fixed">
+        <parent link="base_link"/>
+        <child link="base_footprint"/>
+        <origin xyz="0 0 0" rpy="0 0 0"/>
+    </joint>
+    <link name="base_footprint">
     </link>
     <!-- Chassis -->
