Commit message: rotate lidar

File: description/lidar.xacro (robot description, xacro)
@@ -4,5 +4,5 @@
         <parent link="chassis" />
         <child link="laser_frame" />
-        <origin xyz="0.1 0 0.175" rpy="0 0 0" />
+        <origin xyz="0.1 0 0.175" rpy="0 -${pi/2} 0" />
     </joint>
     <link name="laser_frame">

Commit message: lidar rotate

File: description/lidar.xacro (robot description, xacro)
@@ -4,5 +4,5 @@
         <parent link="chassis" />
         <child link="laser_frame" />
-        <origin xyz="0.1 0 0.175" rpy="0 -${pi/2} 0" />
+        <origin xyz="0.1 0 0.175" rpy="-${pi/2} 0 0" />
     </joint>
     <link name="laser_frame">

Commit message: change dimensions robot

File: description/lidar.xacro (robot description, xacro)
@@ -4,5 +4,5 @@
         <parent link="chassis" />
         <child link="laser_frame" />
-        <origin xyz="0.1 0 0.175" rpy="-${pi/2} 0 0" />
+        <origin xyz="0.2 0 0.17" rpy="0 0 0" />
     </joint>
     <link name="laser_frame">

File: description/robot_core.xacro (robot description, xacro)
@@ -24,5 +24,5 @@
         <parent link="base_link"/>
         <child link="chassis"/>
-        <origin xyz="-0.1 0 0" />
+        <origin xyz="-0.07 0 0" />
     </joint>
     <link name="chassis">
@@ -30,15 +30,15 @@
             <origin xyz="0.15 0 0.075" />
             <geometry>
-                <box size="0.3 0.3 0.15"/>
+                <box size="0.27 0.2 0.17"/>
             </geometry>
             <material name="white"/>
         </visual>
         <collision>
-            <origin xyz="0.15 0 0.075" />
+            <origin xyz="0.10 0 0.075" />
             <geometry>
-                <box size="0.3 0.3 0.15"/>
+                <box size="0.27 0.2 0.17"/>
             </geometry>
         </collision>
-        <xacro:inertial_box mass="0.5" x="0.3" y="0.3" z="0.15" >
+        <xacro:inertial_box mass="0.5" x="0.27" y="0.2" z="0.17" >
             <origin xyz="0.15 0 0.075" rpy="0 0 0"/>
         </xacro:inertial_box>
@@ -48,8 +48,14 @@
     </gazebo>
     <!-- LEFT WHELL LINK -->
+    <!--
+        112 mm is the distance between the center of the wheel and the center of the chassis
+        chassi is 200 mm long
+        wheel is 25 mm long
+        200/2 + 25/2 = 112 mm
+    -->
     <joint name="left_wheel_joint" type="continuous">
         <parent link="base_link"/>
         <child link="left_wheel"/>
-        <origin xyz="0 0.175 0" rpy="-${pi/2} 0 0"/>
+        <origin xyz="0 0.112 0" rpy="-${pi/2} 0 0"/>
         <axis xyz="0 0 1" />
     </joint>
@@ -57,5 +63,5 @@
         <visual>
             <geometry>
-                <cylinder radius="0.05" length="0.04"/>
+                <cylinder radius="0.035" length="0.025"/>
             </geometry>
             <material name="blue"/>
@@ -63,8 +69,8 @@
          <collision>
             <geometry>
-                <cylinder radius="0.05" length="0.04"/>
+                <cylinder radius="0.035" length="0.025"/>
             </geometry>
         </collision>
-        <xacro:inertial_cylinder mass="0.1" length="0.04" radius="0.05" >
+        <xacro:inertial_cylinder mass="0.1" length="0.025" radius="0.035" >
             <origin xyz="0 0 0" rpy="0 0 0"/>
         </xacro:inertial_cylinder>
@@ -77,5 +83,5 @@
         <parent link="base_link"/>
         <child link="right_wheel"/>
-        <origin xyz="0 -0.175 0" rpy="${pi/2} 0 0"/>
+        <origin xyz="0 -0.112 0" rpy="${pi/2} 0 0"/>
         <axis xyz="0 0 -1" />
     </joint>
@@ -83,5 +89,5 @@
         <visual>
             <geometry>
-                <cylinder radius="0.05" length="0.04"/>
+                <cylinder radius="0.035" length="0.025"/>
             </geometry>
             <material name="blue"/>
@@ -89,8 +95,8 @@
         <collision>
             <geometry>
-                <cylinder radius="0.05" length="0.04"/>
+                <cylinder radius="0.035" length="0.025"/>
             </geometry>
         </collision>
-        <xacro:inertial_cylinder mass="0.1" length="0.04" radius="0.05" >
+        <xacro:inertial_cylinder mass="0.1" length="0.025" radius="0.035" >
             <origin xyz="0 0 0" rpy="0 0 0"/>
         </xacro:inertial_cylinder>

File: description/ros2_control.xacro (robot description, xacro)
@@ -29,7 +29,5 @@
         </joint>
     </ros2_control>
-    <!--
-    </ros2_control>
-        <ros2_control name="GazeboSystem" type="system">
+    <!-- <ros2_control name="GazeboSystem" type="system">
         <hardware>
             <plugin>gazebo_ros2_control/GazeboSystem</plugin>
@@ -52,6 +50,5 @@
         </joint>
     </ros2_control>
-    -->
-    <!-- <gazebo>
+    <gazebo>
         <plugin name="gazebo_ros2_control" filename="libgazebo_ros2_control.so">
             <parameters>

Commit message: feat: add nav2

File: description/lidar.xacro (robot description, xacro)
@@ -13,10 +13,10 @@
             <material name="red"/>
         </visual>
-         <collision>
+        <collision>
             <geometry>
                 <cylinder radius="0.05" length="0.04"/>
             </geometry>
         </collision>
-        <xacro:inertial_cylinder mass="0.1" length="0.04" radius="0.05" >
+        <xacro:inertial_cylinder mass="0.1" length="0.04" radius="0.05">
             <origin xyz="0 0 0" rpy="0 0 0"/>
         </xacro:inertial_cylinder>

File: description/robot.urdf.xacro (robot description, xacro)
@@ -1,4 +1,4 @@
 <?xml version="1.0"?>
-<robot xmlns:xacro="http://www.ros.org/wiki/xacro"  name="robot">
+<robot xmlns:xacro="http://www.ros.org/wiki/xacro" name="robot">
     <xacro:arg name="use_ros2_control" default="true" />
     <xacro:arg name="sim_mode" default="false" />
@@ -11,3 +11,4 @@
     </xacro:unless>
     <xacro:include filename="lidar.xacro" />
+    <xacro:include filename="imu.xacro" />
 </robot>
